File: Custom_Teensy_3.1.sch (EAGLE design)
At the start: 37 parts, among them J1 1981584-1, U1 MK20DX256VLH7, U2 TPS61200, U3 MINI54TAN, Y1 32.768KHz, Y2 16Mhz/8pF

Commit message: Removed the I2C connection between MINI54TAN and MK20 as these are not used
As this connection is shown in the official Teensy 3.1 schematics I
have also added it. Paul today stated in the official PJRC forum that
this connection is not used and will never be used. So I removed it.
Connections:
- net SCL: no longer U3.P3.5
- net SDA: no longer U3.P3.4
Changed lines of the file:
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@@
 <net name="SDA" class="0">
 <segment>
-<pinref part="U3" gate="G$1" pin="P3.4"/>
-<wire x1="104.14" y1="-162.56" x2="132.08" y2="-162.56" width="0.1524" layer="91"/>
-<wire x1="132.08" y1="-162.56" x2="132.08" y2="-187.96" width="0.1524" layer="91"/>
-<wire x1="132.08" y1="-187.96" x2="208.28" y2="-187.96" width="0.1524" layer="91"/>
-<wire x1="208.28" y1="-187.96" x2="208.28" y2="-63.5" width="0.1524" layer="91"/>
 <pinref part="U1" gate="G$1" pin="PTB3"/>
-<wire x1="208.28" y1="-63.5" x2="203.2" y2="-63.5" width="0.1524" layer="91"/>
-<wire x1="208.28" y1="-63.5" x2="226.06" y2="-63.5" width="0.1524" layer="91"/>
-<junction x="208.28" y="-63.5"/>
+<wire x1="203.2" y1="-63.5" x2="226.06" y2="-63.5" width="0.1524" layer="91"/>
 <label x="226.06" y="-63.5" size="1.778" layer="95"/>
 </segment>
@@
 <net name="SCL" class="0">
 <segment>
-<pinref part="U3" gate="G$1" pin="P3.5"/>
-<wire x1="104.14" y1="-165.1" x2="129.54" y2="-165.1" width="0.1524" layer="91"/>
-<wire x1="129.54" y1="-165.1" x2="129.54" y2="-190.5" width="0.1524" layer="91"/>
-<wire x1="129.54" y1="-190.5" x2="210.82" y2="-190.5" width="0.1524" layer="91"/>
-<wire x1="210.82" y1="-190.5" x2="210.82" y2="-60.96" width="0.1524" layer="91"/>
 <pinref part="U1" gate="G$1" pin="PTB2"/>
-<wire x1="210.82" y1="-60.96" x2="203.2" y2="-60.96" width="0.1524" layer="91"/>
-<junction x="210.82" y="-60.96"/>
+<wire x1="203.2" y1="-60.96" x2="226.06" y2="-60.96" width="0.1524" layer="91"/>
 <label x="226.06" y="-60.96" size="1.778" layer="95"/>
-<wire x1="210.82" y1="-60.96" x2="226.06" y2="-60.96" width="0.1524" layer="91"/>
 </segment>
 </net>
